File: aux_out/aux_out.kicad_sch (KiCad schematic)
At the start: 9 parts, among them J1 AudioJack2_SwitchT, J2 AudioJack2_SwitchT, J3 AudioJack3

Commit message: Layout aux module
Parts:
- J1, J2: footprint (none) -> custom_fp:PJ398SM
- J3: footprint (none) -> custom_fp:PJ366ST
- R1, R2, R3, R4, R5, R6: footprint (none) -> Resistor_SMD:R_0603_1608Metric
Changed lines of the file:
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@@
       (effects (font (size 1.27 1.27)) (justify left))
     )
-    (property "Footprint" "" (at 122.682 67.31 90)
+    (property "Footprint" "Resistor_SMD:R_0603_1608Metric" (at 122.682 67.31 90)
       (effects (font (size 1.27 1.27)) hide)
     )
@@
       (effects (font (size 1.27 1.27)))
     )
-    (property "Footprint" "" (at 129.54 94.488 90)
+    (property "Footprint" "Resistor_SMD:R_0603_1608Metric" (at 129.54 94.488 90)
       (effects (font (size 1.27 1.27)) hide)
     )
@@
       (effects (font (size 1.27 1.27)) (justify right))
     )
-    (property "Footprint" "" (at 161.29 73.66 0)
+    (property "Footprint" "custom_fp:PJ366ST" (at 161.29 73.66 0)
       (effects (font (size 1.27 1.27)) hide)
     )
@@
       (effects (font (size 1.27 1.27)))
     )
-    (property "Footprint" "" (at 96.52 92.71 0)
+    (property "Footprint" "custom_fp:PJ398SM" (at 96.52 92.71 0)
       (effects (font (size 1.27 1.27)) hide)
     )
@@
       (effects (font (size 1.27 1.27)))
     )
-    (property "Footprint" "" (at 119.38 64.008 90)
+    (property "Footprint" "Resistor_SMD:R_0603_1608Metric" (at 119.38 64.008 90)
       (effects (font (size 1.27 1.27)) hide)
     )
@@
       (effects (font (size 1.27 1.27)))
     )
-    (property "Footprint" "" (at 119.38 94.488 90)
+    (property "Footprint" "Resistor_SMD:R_0603_1608Metric" (at 119.38 94.488 90)
       (effects (font (size 1.27 1.27)) hide)
     )
@@
       (effects (font (size 1.27 1.27)))
     )
-    (property "Footprint" "" (at 129.54 64.008 90)
+    (property "Footprint" "Resistor_SMD:R_0603_1608Metric" (at 129.54 64.008 90)
       (effects (font (size 1.27 1.27)) hide)
     )
@@
       (effects (font (size 1.27 1.27)))
     )
-    (property "Footprint" "" (at 96.52 62.23 0)
+    (property "Footprint" "custom_fp:PJ398SM" (at 96.52 62.23 0)
       (effects (font (size 1.27 1.27)) hide)
     )
@@
       (effects (font (size 1.27 1.27)) (justify left))
     )
-    (property "Footprint" "" (at 122.682 97.79 90)
-      (effects (font (size 1.27 1.27)) hide)
-    )
+    (property "Footprint" "Resistor_SMD:R_0603_1608Metric" (at 122.682 97.79 90)
+      (effects (font (size 1.27 1.27)) hide)
+    )
