File: PATCH_BAY/PATCH_BAY.kicad_sch (KiCad schematic)
At the start: 7 parts, among them J1 AudioJack2_SwitchT, J2 AudioJack2_SwitchT, J3 AudioJack2_SwitchT, J4 AudioJack2_SwitchT, J5 AudioJack2_SwitchT, J6 AudioJack2_SwitchT, J7 Conn_01x12_Pin

Commit message: Layout patch bay
Parts:
- J1, J2, J3, J4, J5, J6: footprint (none) -> Custom_FP:PJ398SM
- J7: value Conn_01x12_Pin -> Conn_01x10_Pin; footprint (none) -> Connector_PinHeader_2.54mm:PinHeader_2x05_P2.54mm_Vertical_SMD; symbol Connector:Conn_01x12_Pin -> Connector:Conn_01x10_Pin
Connections:
- net GND: now also J7.1 (Pin_1), J7.9 (Pin_9); no longer J7.12 (Pin_12), J7.4 (Pin_4), J7.6 (Pin_6), J7.8 (Pin_8)
- net at J4.T: now also J7.6 (Pin_6); no longer J7.7 (Pin_7)
- net at J1.T: now also J7.3 (Pin_3); no longer J7.1 (Pin_1)
- net at J6.T: now also J7.8 (Pin_8); no longer J7.11 (Pin_11)
- net at J2.T: now also J7.4 (Pin_4); no longer J7.3 (Pin_3)
- net at J5.T: now also J7.7 (Pin_7); no longer J7.9 (Pin_9)
