File: PATCH_BAY/PATCH_BAY.kicad_pcb (KiCad board)
At the start: 2 copper layers, 40.2 x 22.5 mm, 7 parts, among them J1 AudioJack2_SwitchT, J2 AudioJack2_SwitchT, J3 AudioJack2_SwitchT, J4 AudioJack2_SwitchT, J5 AudioJack2_SwitchT, J6 AudioJack2_SwitchT, J7 Conn_01x10_Pin

Commit message: Add PATCH front panel
Other:
- board text added: "Patch bay"
Changed lines of the file:
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@@
 		(at 129.75 60.5 180)
 		(property "Reference" "J1"
-			(at 0 -7 360)
+			(at 0 -7 0)
 			(layer "F.SilkS")
 			(effects
@@
 		)
 		(property "Value" "AudioJack2_SwitchT"
-			(at 0 -8.25 360)
+			(at 0 -8.25 0)
 			(layer "F.Fab")
 			(effects
@@
 		)
 		(property "Footprint" "Custom_FP:PJ398SM"
-			(at 0 0 360)
+			(at 0 0 0)
 			(layer "F.Fab")
 			(hide yes)
@@
 		)
 		(property "Datasheet" ""
-			(at 0 0 360)
+			(at 0 0 0)
 			(layer "F.Fab")
 			(hide yes)
@@
 		)
 		(property "Description" ""
-			(at 0 0 360)
+			(at 0 0 0)
 			(layer "F.Fab")
 			(hide yes)
@@
 		(at 160.5 60.5 180)
 		(property "Reference" "J6"
-			(at 0 -6.75 360)
+			(at 0 -6.75 0)
 			(layer "F.SilkS")
 			(effects
@@
 		)
 		(property "Value" "AudioJack2_SwitchT"
-			(at 0 -8.25 360)
+			(at 0 -8.25 0)
 			(layer "F.Fab")
 			(effects
@@
 		)
 		(property "Footprint" "Custom_FP:PJ398SM"
-			(at 0 0 360)
+			(at 0 0 0)
 			(layer "F.Fab")
 			(hide yes)
@@
 		)
 		(property "Datasheet" ""
-			(at 0 0 360)
+			(at 0 0 0)
 			(layer "F.Fab")
 			(hide yes)
@@
 		)
 		(property "Description" ""
-			(at 0 0 360)
+			(at 0 0 0)
 			(layer "F.Fab")
 			(hide yes)
@@
 		(layer "Edge.Cuts")
 	)
+	(gr_text "Patch bay"
+		(at 161.5 61.5 0)
+		(layer "B.SilkS")
+		(effects
+			(font
+				(size 1 1)
+				(thickness 0.15)
+			)
+			(justify left bottom mirror)
+		)
+	)
 	(segment
