File: MULT/MULT.kicad_sch (KiCad schematic)
At the start: 8 parts, among them J1 AudioJack2_SwitchT, J2 AudioJack2_SwitchT, J3 AudioJack2_SwitchT, J4 AudioJack2_SwitchT, J5 AudioJack2_SwitchT, J6 AudioJack2_SwitchT, J7 AudioJack2_SwitchT, J8 AudioJack2_SwitchT

Commit message: Layout mult
Parts:
- J1, J2, J3, J4, J5, J6, J7, J8: footprint (none) -> Custom_FP:PJ398SM
Changed lines of the file:
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@@
 			)
 		)
-		(property "Footprint" ""
+		(property "Footprint" "Custom_FP:PJ398SM"
 			(at 98.425 71.12 0)
 			(effects
@@
 			)
 		)
-		(property "Footprint" ""
+		(property "Footprint" "Custom_FP:PJ398SM"
 			(at 98.425 86.36 0)
 			(effects
@@
 			)
 		)
-		(property "Footprint" ""
+		(property "Footprint" "Custom_FP:PJ398SM"
 			(at 63.5 102.235 0)
 			(effects
@@
 			)
 		)
-		(property "Footprint" ""
+		(property "Footprint" "Custom_FP:PJ398SM"
 			(at 63.5 55.88 0)
 			(effects
@@
 			)
 		)
-		(property "Footprint" ""
+		(property "Footprint" "Custom_FP:PJ398SM"
 			(at 98.425 55.88 0)
 			(effects
@@
 			)
 		)
-		(property "Footprint" ""
+		(property "Footprint" "Custom_FP:PJ398SM"
 			(at 98.425 102.235 0)
 			(effects
@@
 			)
 		)
-		(property "Footprint" ""
+		(property "Footprint" "Custom_FP:PJ398SM"
 			(at 98.425 117.475 0)
 			(effects
@@
 			)
 		)
-		(property "Footprint" ""
+		(property "Footprint" "Custom_FP:PJ398SM"
 			(at 98.425 132.715 0)
 			(effects
