File: CLIP/CLIP.kicad_sch (KiCad schematic)
At the start: 19 parts, among them J1 AudioJack2_SwitchT, J2 AudioJack2_SwitchT, J3 AudioJack2_SwitchT, J4 AudioJack2_SwitchT

Commit message: Layout CLIP
Parts:
- D1, D2, D3, D4, D5, D6, D7, D8: value D -> 1N4148; footprint (none) -> Diode_SMD:D_SOD-323_HandSoldering
- D10, D9: value 3v3 zener -> BZX384C3V3-E3-08; footprint (none) -> Diode_SMD:D_SOD-323_HandSoldering
- D11, D12: value 2v zener -> BZT52C2V0S; footprint (none) -> Diode_SMD:D_SOD-323_HandSoldering
- J1, J2, J3, J4: footprint (none) -> Custom_FP:PJ398SM
- R1, R2, R3: footprint (none) -> Resistor_SMD:R_0603_1608Metric
Other:
- moved on the sheet: D1
