File: CLIP/CLIP.kicad_pcb (KiCad board)
At the start: 2 copper layers, 30 x 22.5 mm, 19 parts, among them J1 AudioJack2_SwitchT, J2 AudioJack2_SwitchT, J3 AudioJack2_SwitchT, J4 AudioJack2_SwitchT

Commit message: Add CLIPPER front panel
Other:
- board text added: "Passive CLIPPER"
Changed lines of the file:
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@@
 		(at 139.25 87.03)
 		(property "Reference" "J3"
-			(at 0 -6.75 360)
+			(at 0 -6.75 0)
 			(layer "F.SilkS")
 			(effects
@@
 		)
 		(property "Value" "AudioJack2_SwitchT"
-			(at 0 -8.25 360)
+			(at 0 -8.25 0)
 			(layer "F.Fab")
 			(effects
@@
 		)
 		(property "Footprint" "Custom_FP:PJ398SM"
-			(at 0 0 360)
+			(at 0 0 0)
 			(layer "F.Fab")
 			(hide yes)
@@
 		)
 		(property "Datasheet" ""
-			(at 0 0 360)
+			(at 0 0 0)
 			(layer "F.Fab")
 			(hide yes)
@@
 		)
 		(property "Description" "Audio Jack, 2 Poles (Mono / TS), Switched T Pole (Normalling)"
-			(at 0 0 360)
+			(at 0 0 0)
 			(layer "F.Fab")
 			(hide yes)
@@
 		(tags "resistor")
 		(property "Reference" "R3"
-			(at 0 1.43 360)
+			(at 0 1.43 0)
 			(layer "B.SilkS")
 			(effects
@@
 		)
 		(property "Value" "10k"
-			(at 0 -1.43 360)
+			(at 0 -1.43 0)
 			(layer "B.Fab")
 			(effects
@@
 		)
 		(fp_text user "${REFERENCE}"
-			(at 0 0 360)
+			(at 0 0 0)
 			(layer "B.Fab")
 			(effects
@@
 		(tags "SOD-323")
 		(property "Reference" "D4"
-			(at 0 -1.75 360)
+			(at 0 -1.75 0)
 			(layer "B.SilkS")
 			(effects
@@
 		)
 		(property "Value" "1N4148"
-			(at 0.1 -1.9 360)
+			(at 0.1 -1.9 0)
 			(layer "B.Fab")
 			(effects
@@
 		)
 		(fp_text user "${REFERENCE}"
-			(at 0 1.85 360)
+			(at 0 1.85 0)
 			(layer "B.Fab")
 			(effects
@@
 		(tags "SOD-323")
 		(property "Reference" "D2"
-			(at 0 -1.75 360)
+			(at 0 -1.75 0)
 			(layer "B.SilkS")
 			(effects
@@
 		)
 		(property "Value" "1N4148"
-			(at 0.1 -1.9 360)
+			(at 0.1 -1.9 0)
 			(layer "B.Fab")
 			(effects
@@
 		)
 		(fp_text user "${REFERENCE}"
-			(at 0 1.85 360)
+			(at 0 1.85 0)
 			(layer "B.Fab")
 			(effects
@@
 		(tags "SOD-323")
 		(property "Reference" "D9"
-			(at 0 1.85 360)
+			(at 0 1.85 0)
 			(layer "B.SilkS")
 			(effects
@@
 		)
 		(property "Value" "BZX384C3V3-E3-08"
-			(at 0.1 -1.9 360)
+			(at 0.1 -1.9 0)
 			(layer "B.Fab")
 			(effects
@@
 		)
 		(fp_text user "${REFERENCE}"
-			(at 0 1.85 360)
+			(at 0 1.85 0)
 			(layer "B.Fab")
 			(effects
@@
 		(tags "SOD-323")
 		(property "Reference" "D7"
-			(at 0.25 -1.75 360)
+			(at 0.25 -1.75 0)
 			(layer "B.SilkS")
 			(effects
@@
 		)
 		(property "Value" "1N4148"
-			(at 0.1 -1.9 360)
+			(at 0.1 -1.9 0)
 			(layer "B.Fab")
 			(effects
@@
 		)
 		(fp_text user "${REFERENCE}"
-			(at 0 1.85 360)
+			(at 0 1.85 0)
 			(layer "B.Fab")
 			(effects
@@
 		(tags "SOD-323")
 		(property "Reference" "D10"
-			(at 0.75 -1.75 360)
+			(at 0.75 -1.75 0)
 			(layer "B.SilkS")
 			(effects
@@
 		)
 		(property "Value" "BZX384C3V3-E3-08"
-			(at 0.1 -1.9 360)
+			(at 0.1 -1.9 0)
 			(layer "B.Fab")
 			(effects
@@
 		)
 		(fp_text user "${REFERENCE}"
-			(at 0 1.85 360)
+			(at 0 1.85 0)
 			(layer "B.Fab")
 			(effects
@@
 		(tags "SOD-323")
 		(property "Reference" "D1"
-			(at 0 -1.75 360)
+			(at 0 -1.75 0)
 			(layer "B.SilkS")
 			(effects
@@
 		)
 		(property "Value" "1N4148"
-			(at 0.1 -1.9 360)
+			(at 0.1 -1.9 0)
 			(layer "B.Fab")
 			(effects
@@
 		)
 		(fp_text user "${REFERENCE}"
-			(at 0 1.85 360)
+			(at 0 1.85 0)
 			(layer "B.Fab")
 			(effects
@@
 		(tags "resistor")
 		(property "Reference" "R2"
-			(at 0 -1.5 360)
+			(at 0 -1.5 0)
 			(layer "B.SilkS")
 			(effects
@@
 		)
 		(property "Value" "10k"
-			(at 0 -1.43 360)
+			(at 0 -1.43 0)
 			(layer "B.Fab")
 			(effects
@@
 		)
 		(fp_text user "${REFERENCE}"
-			(at 0 0 360)
+			(at 0 0 0)
 			(layer "B.Fab")
 			(effects
@@
 		(tags "SOD-323")
 		(property "Reference" "D3"
-			(at 0 -1.75 360)
+			(at 0 -1.75 0)
 			(layer "B.SilkS")
 			(effects
@@
 		)
 		(property "Value" "1N4148"
-			(at 0.1 -1.9 360)
+			(at 0.1 -1.9 0)
 			(layer "B.Fab")
 			(effects
@@
 		)
 		(fp_text user "${REFERENCE}"
-			(at 0 1.85 360)
+			(at 0 1.85 0)
 			(layer "B.Fab")
 			(effects
@@
 		(layer "Edge.Cuts")
 	)
+	(gr_text "Passive\nCLIPPER"
+		(at 149.5 96.25 0)
+		(layer "B.SilkS")
+		(effects
+			(font
+				(size 1 1)
+				(thickness 0.1)
+			)
+			(justify bottom mirror)
+		)
+	)
 	(segment
