File: AND_FRONT/AND_FRONT.kicad_pcb (KiCad board)
At the start: 2 copper layers, 20.2 x 43.2 mm, 5 parts, among them J1 Screw_Terminal_01x01, J2 Screw_Terminal_01x01, J3 Screw_Terminal_01x01, J4 Screw_Terminal_01x01, J5 Screw_Terminal_01x01

Commit message: Finalize modules
Other:
- board text added: "JLCJLCJLCJLC"
Changed lines of the file:
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@@
 			(plot_on_all_layers_selection 0x0000000_00000000)
 			(disableapertmacros no)
-			(usegerberextensions no)
-			(usegerberattributes yes)
-			(usegerberadvancedattributes yes)
-			(creategerberjobfile yes)
+			(usegerberextensions yes)
+			(usegerberattributes no)
+			(usegerberadvancedattributes no)
+			(creategerberjobfile no)
 			(dashed_line_dash_ratio 12.000000)
 			(dashed_line_gap_ratio 3.000000)
@@
 			(psa4output no)
 			(plotreference yes)
-			(plotvalue yes)
+			(plotvalue no)
 			(plotfptext yes)
 			(plotinvisibletext no)
 			(sketchpadsonfab no)
-			(subtractmaskfromsilk no)
+			(subtractmaskfromsilk yes)
 			(outputformat 1)
 			(mirror no)
-			(drillshape 1)
+			(drillshape 0)
 			(scaleselection 1)
-			(outputdirectory "")
+			(outputdirectory "out/")
 		)
 	)
@@
 	)
 	(gr_line
-		(start 107.05 97.25)
-		(end 105.35 97.25)
+		(start 107.25 97.25)
+		(end 105.5 97.25)
 		(stroke
 			(width 0.3)
@@
 	)
 	(gr_line
-		(start 105.35 95.95)
-		(end 105.35 93.35)
+		(start 105.5 95.75)
+		(end 105.5 93.35)
 		(stroke
 			(width 0.3)
@@
 	)
 	(gr_rect
-		(start 107.05 95.45)
-		(end 108.9 97.75)
+		(start 107 95)
+		(end 108.9 98)
 		(stroke
 			(width 0.1)
@@
 	)
 	(gr_line
-		(start 105.35 97.25)
-		(end 105.35 99.95)
+		(start 105.5 97.25)
+		(end 105.5 99.95)
 		(stroke
 			(width 0.3)
@@
 	)
 	(gr_line
-		(start 107.05 95.95)
-		(end 105.35 95.95)
+		(start 107.25 95.75)
+		(end 105.5 95.75)
 		(stroke
 			(width 0.3)
@@
 	)
 	(gr_circle
-		(center 108.9 96.6)
-		(end 110.05 96.6)
+		(center 108.9 96.5)
+		(end 110.4 96.5)
 		(stroke
 			(width 0.1)
@@
 	)
 	(gr_line
-		(start 110.05 96.6)
-		(end 111.9 96.6)
+		(start 110.25 96.5)
+		(end 112 96.5)
 		(stroke
 			(width 0.3)
@@
 		(layer "User.2")
 	)
+	(gr_text "JLCJLCJLCJLC"
+		(at 116 110.75 0)
+		(layer "B.SilkS")
+		(effects
+			(font
+				(size 1 1)
+				(thickness 0.1)
+			)
+			(justify left bottom mirror)
+		)
+	)
 	(gr_text "AND"
-		(at 107.85 84.3 0)
+		(at 111.25 83.25 0)
 		(layer "F.Mask")
 		(effects
@@
 				(thickness 0.15)
 			)
-			(justify left bottom)
+			(justify bottom)
 		)
 	)
@@
 		(layers "F&B.Cu")
 		(hatch edge 0.5)
-		(connect_pads
+		(connect_pads yes
 			(clearance 0.5)
 		)
