File: PATCH_FRONT/PATCH_FRONT.kicad_pcb (KiCad board)
At the start: 2 copper layers, 40.6 x 43.2 mm, 10 parts, among them J1 Screw_Terminal_01x01, J10 Screw_Terminal_01x01, J2 Screw_Terminal_01x01, J3 Screw_Terminal_01x01, J4 Screw_Terminal_01x01, J5 Screw_Terminal_01x01, J6 Screw_Terminal_01x01, J7 Screw_Terminal_01x01, J8 Screw_Terminal_01x01, J9 Screw_Terminal_01x01

Commit message: Finalize modules
Other:
- board text added: "JLCJLCJLCJLC"
- board text added: "PORTAL"
- board text removed: "Portal"
Changed lines of the file:
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@@
 			(plot_on_all_layers_selection 0x0000000_00000000)
 			(disableapertmacros no)
-			(usegerberextensions no)
-			(usegerberattributes yes)
-			(usegerberadvancedattributes yes)
-			(creategerberjobfile yes)
+			(usegerberextensions yes)
+			(usegerberattributes no)
+			(usegerberadvancedattributes no)
+			(creategerberjobfile no)
 			(dashed_line_dash_ratio 12.000000)
 			(dashed_line_gap_ratio 3.000000)
@@
 			(psa4output no)
 			(plotreference yes)
-			(plotvalue yes)
+			(plotvalue no)
 			(plotfptext yes)
 			(plotinvisibletext no)
 			(sketchpadsonfab no)
-			(subtractmaskfromsilk no)
+			(subtractmaskfromsilk yes)
 			(outputformat 1)
 			(mirror no)
-			(drillshape 1)
+			(drillshape 0)
 			(scaleselection 1)
-			(outputdirectory "")
+			(outputdirectory "out/")
 		)
 	)
@@
 		(layer "User.2")
 	)
-	(gr_text "Portal"
-		(at 115.85 83.65 0)
+	(gr_text "JLCJLCJLCJLC"
+		(at 125 110.75 0)
+		(layer "B.SilkS")
+		(effects
+			(font
+				(size 1 1)
+				(thickness 0.1)
+			)
+			(justify left bottom mirror)
+		)
+	)
+	(gr_text "PORTAL"
+		(at 120.25 83 0)
 		(layer "F.Mask")
 		(effects
 			(font
 				(size 2 2)
-				(thickness 0.3)
-				(bold yes)
-			)
-			(justify left bottom)
-		)
-	)
+				(thickness 0.15)
+			)
+			(justify bottom)
+		)
+	)
