File: RECT/RECT.kicad_pcb (KiCad board)
At the start: 2 copper layers, 30 x 22.5 mm, 10 parts, among them J1 AudioJack2_SwitchT, J2 AudioJack2_SwitchT, J3 AudioJack2_SwitchT, J4 AudioJack2_SwitchT, Q1 BSS84, Q2 BSS84, Q3 2N7002, Q4 2N7002

Commit message: Fix rectifier DRC
Parts:
- R1, R2: value 100k -> 1M

Commit message: Add RECT front panel
Other:
- board text added: "Passive RECTIFIER"
Changed lines of the file:
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@@
 		(layer "Edge.Cuts")
+	)
+	(gr_text "Passive\nRECTIFIER"
+		(at 129.6 63 0)
+		(layer "B.SilkS")
+		(effects
+			(font
+				(size 1 1)
+				(thickness 0.15)
+			)
+			(justify bottom mirror)
+		)
 	)
 	(gr_text "MIN OUT"
