File: RECT_FRONT/RECT_FRONT.kicad_pcb (KiCad board)
At the start: 2 copper layers, 30.5 x 43.2 mm, 8 parts, among them J1 Screw_Terminal_01x01, J2 Screw_Terminal_01x01, J3 Screw_Terminal_01x01, J4 Screw_Terminal_01x01, J5 Screw_Terminal_01x01, J6 Screw_Terminal_01x01, J7 Screw_Terminal_01x01, J8 Screw_Terminal_01x01

Commit message: Finalize modules
Other:
- board text added: "JLCJLCJLCJLC"
Changed lines of the file:
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@@
 			(plot_on_all_layers_selection 0x0000000_00000000)
 			(disableapertmacros no)
-			(usegerberextensions no)
-			(usegerberattributes yes)
-			(usegerberadvancedattributes yes)
-			(creategerberjobfile yes)
+			(usegerberextensions yes)
+			(usegerberattributes no)
+			(usegerberadvancedattributes no)
+			(creategerberjobfile no)
 			(dashed_line_dash_ratio 12.000000)
 			(dashed_line_gap_ratio 3.000000)
@@
 			(psa4output no)
 			(plotreference yes)
-			(plotvalue yes)
+			(plotvalue no)
 			(plotfptext yes)
 			(plotinvisibletext no)
 			(sketchpadsonfab no)
-			(subtractmaskfromsilk no)
+			(subtractmaskfromsilk yes)
 			(outputformat 1)
 			(mirror no)
-			(drillshape 1)
+			(drillshape 0)
 			(scaleselection 1)
-			(outputdirectory "")
+			(outputdirectory "out/")
 		)
 	)
@@
 	)
 	(gr_line
+		(start 118.75 91.75)
+		(end 117.5 88.5)
+		(stroke
+			(width 0.3)
+			(type default)
+		)
+		(layer "F.Mask")
+	)
+	(gr_line
+		(start 118.75 101.25)
+		(end 117.5 104.5)
+		(stroke
+			(width 0.3)
+			(type default)
+		)
+		(layer "F.Mask")
+	)
+	(gr_line
+		(start 103.5 99.75)
+		(end 101.25 97.5)
+		(stroke
+			(width 0.3)
+			(type default)
+		)
+		(layer "F.Mask")
+	)
+	(gr_line
+		(start 103.5 87.25)
+		(end 102.5 87.25)
+		(stroke
+			(width 0.3)
+			(type default)
+		)
+		(layer "F.Mask")
+	)
+	(gr_line
+		(start 103.5 87.25)
+		(end 101.25 85)
+		(stroke
+			(width 0.3)
+			(type default)
+		)
+		(layer "F.Mask")
+	)
+	(gr_line
+		(start 103.5 87.25)
+		(end 103.5 86.25)
+		(stroke
+			(width 0.3)
+			(type default)
+		)
+		(layer "F.Mask")
+	)
+	(gr_line
+		(start 103.5 99.75)
+		(end 102.5 99.75)
+		(stroke
+			(width 0.3)
+			(type default)
+		)
+		(layer "F.Mask")
+	)
+	(gr_line
+		(start 103.5 99.75)
+		(end 103.5 98.75)
+		(stroke
+			(width 0.3)
+			(type default)
+		)
+		(layer "F.Mask")
+	)
+	(gr_line
+		(start 117.5 104.5)
+		(end 116.25 101.25)
+		(stroke
+			(width 0.3)
+			(type default)
+		)
+		(layer "F.Mask")
+	)
+	(gr_line
+		(start 117.5 88.5)
+		(end 116.25 91.75)
+		(stroke
+			(width 0.3)
+			(type default)
+		)
+		(layer "F.Mask")
+	)
+	(gr_line
 		(start 99.85 75)
 		(end 99.85 118.25)
@@
 		(layer "User.2")
 	)
+	(gr_text "JLCJLCJLCJLC"
+		(at 119.5 110.5 0)
+		(layer "B.SilkS")
+		(effects
+			(font
+				(size 1 1)
+				(thickness 0.1)
+			)
+			(justify left bottom mirror)
+		)
+	)
 	(gr_text "RECTIFY"
-		(at 109.1 84.5 0)
+		(at 109.1 83 0)
 		(layer "F.Mask")
 		(effects
