File: XOR_FRONT/XOR_FRONT.kicad_pcb (KiCad board)
At the start: 2 copper layers, 20.2 x 43.2 mm, 5 parts, among them J1 Screw_Terminal_01x01, J2 Screw_Terminal_01x01, J3 Screw_Terminal_01x01, J4 Screw_Terminal_01x01, J5 Screw_Terminal_01x01

Commit message: Finalize modules
Other:
- board text added: "JLCJLCJLCJLC"
Changed lines of the file:
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@@
 			(plot_on_all_layers_selection 0x0000000_00000000)
 			(disableapertmacros no)
-			(usegerberextensions no)
-			(usegerberattributes yes)
-			(usegerberadvancedattributes yes)
-			(creategerberjobfile yes)
+			(usegerberextensions yes)
+			(usegerberattributes no)
+			(usegerberadvancedattributes no)
+			(creategerberjobfile no)
 			(dashed_line_dash_ratio 12.000000)
 			(dashed_line_gap_ratio 3.000000)
@@
 			(psa4output no)
 			(plotreference yes)
-			(plotvalue yes)
+			(plotvalue no)
 			(plotfptext yes)
 			(plotinvisibletext no)
 			(sketchpadsonfab no)
-			(subtractmaskfromsilk no)
+			(subtractmaskfromsilk yes)
 			(outputformat 1)
 			(mirror no)
-			(drillshape 1)
+			(drillshape 0)
 			(scaleselection 1)
-			(outputdirectory "")
+			(outputdirectory "out/")
 		)
 	)
@@
 		)
 	)
+	(gr_arc
+		(start 108.75 95)
+		(mid 109.961673 95.486004)
+		(end 110.857963 96.435222)
+		(stroke
+			(width 0.1)
+			(type default)
+		)
+		(layer "F.Mask")
+	)
+	(gr_arc
+		(start 107 95.000001)
+		(mid 107.92705 96.5)
+		(end 107 97.999999)
+		(stroke
+			(width 0.1)
+			(type default)
+		)
+		(layer "F.Mask")
+	)
+	(gr_arc
+		(start 106.5 95.000001)
+		(mid 107.42705 96.5)
+		(end 106.5 97.999999)
+		(stroke
+			(width 0.1)
+			(type default)
+		)
+		(layer "F.Mask")
+	)
+	(gr_line
+		(start 108 95.75)
+		(end 105.5 95.75)
+		(stroke
+			(width 0.3)
+			(type default)
+		)
+		(layer "F.Mask")
+	)
+	(gr_line
+		(start 108 97.25)
+		(end 105.5 97.25)
+		(stroke
+			(width 0.3)
+			(type default)
+		)
+		(layer "F.Mask")
+	)
+	(gr_line
+		(start 105.5 97.25)
+		(end 105.5 99.75)
+		(stroke
+			(width 0.3)
+			(type default)
+		)
+		(layer "F.Mask")
+	)
+	(gr_poly
+		(pts
+			(xy 108.75 95) (xy 109.961673 95.486004) (xy 110.89066 96.508946) (xy 109.988317 97.495647) (xy 108.75 98)
+		)
+		(stroke
+			(width 0.1)
+			(type solid)
+		)
+		(fill solid)
+		(layer "F.Mask")
+	)
+	(gr_rect
+		(start 108.000001 95)
+		(end 108.75 98)
+		(stroke
+			(width 0.1)
+			(type solid)
+		)
+		(fill solid)
+		(layer "F.Mask")
+	)
+	(gr_line
+		(start 105.5 95.75)
+		(end 105.5 93.25)
+		(stroke
+			(width 0.3)
+			(type default)
+		)
+		(layer "F.Mask")
+	)
+	(gr_arc
+		(start 110.89066 96.508946)
+		(mid 109.988317 97.495647)
+		(end 108.75 98)
+		(stroke
+			(width 0.1)
+			(type default)
+		)
+		(layer "F.Mask")
+	)
+	(gr_line
+		(start 110.89066 96.508946)
+		(end 112.75 96.5)
+		(stroke
+			(width 0.3)
+			(type default)
+		)
+		(layer "F.Mask")
+	)
+	(gr_poly
+		(pts
+			(xy 107.000001 95.000001) (xy 108.250001 95) (xy 108.250001 98) (xy 107.000001 97.999999) (xy 107.500001 97.75)
+			(xy 108.000001 96.75) (xy 108.000001 96.25) (xy 107.500001 95.25)
+		)
+		(stroke
+			(width 0.1)
+			(type solid)
+		)
+		(fill solid)
+		(layer "F.Mask")
+	)
 	(gr_line
 		(start 100 75)
@@
 		(layer "User.2")
 	)
+	(gr_text "JLCJLCJLCJLC"
+		(at 115.5 110.75 0)
+		(layer "B.SilkS")
+		(effects
+			(font
+				(size 1 1)
+				(thickness 0.1)
+			)
+			(justify left bottom mirror)
+		)
+	)
 	(gr_text "XOR"
-		(at 107.2 84.25 0)
+		(at 108 83 0)
 		(layer "F.Mask")
 		(effects
